File: TurtleSensor.kicad_pcb (KiCad board)
At the start: 2 copper layers, 72 x 72 mm, 11 parts, among them IC1 ATMEGA328-P, J1 ISPConnector, U1 HTU21DBreakout, U2 W25Q32FlashBreakout

Commit message: swapped layers and added programming header
Parts:
- added C2: 0.1uF, Capacitors_ThroughHole:C_Disc_D3_P2.5, F.Cu at (122.0, 92.0)
- added J2: FTDIConnector, Socket_Strips:Socket_Strip_Angled_1x06, F.Cu at (115.0, 98.0)
- moved BT1 12.5 mm to (104.0, 109.0)
Connections:
- IC1 pad 2: Net-(IC1-Pad2) -> /RX
- IC1 pad 3: Net-(IC1-Pad3) -> /TX
Routing:
- net GND: track 155.4 -> 181.0 mm
- net /TX: track 0.00 -> 23.8 mm
- net Net-(C2-Pad1): track 0.00 -> 22.2 mm
- net /RX: track 0.00 -> 20.3 mm
- net +BATT: track 109.6 -> 126.6 mm
- net /~RST: track 56.1 -> 68.3 mm
- net (no net): track 0.00 -> 0.54 mm
